File: project/Power.kicad_sch (KiCad schematic)
At the start: 20 parts, among them IC101 nPM1300-QEXX, X101 BATTERY

Commit message: PCB: Remove BME688 and USB switch
- Implement #106
- Remove USB switch and the required components

Signed-off-by: Daniel Kampert <danielkampert@kampis-elektroecke.de>
Other:
- title: ZSWatch v2 -> ZSWatch v3
Changed lines of the file:
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@@
 	(paper "A4")
 	(title_block
-		(title "ZSWatch v2")
-		(date "2024-07-23")
-		(rev "6")
+		(title "ZSWatch v3")
+		(date "2025-05-05")
+		(rev "1")
 		(company "github.com/jakkra/ZSWatch-HW")
 	)
