File: hardware/MCU.kicad_sch (KiCad schematic)
At the start: 33 parts, among them IC302 FAN5622SX, IC303 MX25U51245GZ4I00, IC305 NTS0104GU12, IC306 DRV2603RUNT, IC307 RV-8263-C8, M301 NORA-B106, M302 Vibrator DC Motor, Q301 BC817W, Q302 PMZ550UNEYL, Q303 PMZ550UNEYL, X302 GC9A01A_CST816S, X303 M+, X304 M-

Commit message: KiBot: Enhance KiBot configuration
- Implement #110
- Implement #109
- Add refresh for PCB specifications
- Add refresh for stackup

Signed-off-by: Daniel Kampert <danielkampert@kampis-elektroecke.de>
Parts:
- BZ301: Mfr. CUI Devices -> (none); Mfr. No. CMT-322-65-SMT-TR -> (none); Order Number 490-CMT-322-65-SMTTR -> (none); manf (none) -> CUI Devices; manf# (none) -> CMT-322-65-SMT-TR; mouser# (none) -> 490-CMT-322-65-SMTTR
- C301: Mfr. KYOCERA AVX -> (none); Mfr. No. 0603YC105JAT2A -> (none); Order Number 581-0603YC105JAT2A -> (none); manf (none) -> KYOCERA AVX; manf# (none) -> 0603YC105JAT2A; mouser# (none) -> 581-0603YC105JAT2A
- C302, C304, C305, C306: Mfr. KYOCERA AVX -> (none); Mfr. No. 06035C104KAT2A -> (none); Order Number 581-06035C104KAT2A -> (none); manf (none) -> KYOCERA AVX; manf# (none) -> 06035C104KAT2A; mouser# (none) -> 581-06035C104KAT2A
- C307: Mfr. KYOCERA AVX -> (none); Mfr. No. 04025C104KAT2A -> (none); Order Number 581-04025C104KAT2A -> (none); manf (none) -> KYOCERA AVX; manf# (none) -> 04025C104KAT2A; mouser# (none) -> 581-04025C104KAT2A
- D301: Mfr. Taiwan Semiconductor -> (none); Mfr. No. BAS316 RRG -> (none); Order Number 821-BAS316RRG -> (none); manf (none) -> Taiwan Semiconductor; manf# (none) -> BAS316 RRG; mouser# (none) -> 821-BAS316RRG
- IC302: Mfr. onsemi / Fairchild -> (none); Mfr. No. FAN5622SX -> (none); Order Number 512-FAN5622SX -> (none); manf (none) -> onsemi / Fairchild; manf# (none) -> FAN5622SX; mouser# (none) -> 512-FAN5622SX
- IC303: Mfr. Macronix -> (none); Mfr. No. MX25U51245GZ4I00 -> (none); Order Number 95-25U51245GZ4I00T -> (none); manf (none) -> Macronix; manf# (none) -> MX25U51245GZ4I00; mouser# (none) -> 95-25U51245GZ4I00T
- IC305: Mfr. NXP Semiconductors -> (none); Mfr. No. NTS0104GU12,115 -> (none); Order Number 771-NTS0104GU12115 -> (none); manf (none) -> NXP Semiconductors; manf# (none) -> NTS0104GU12,115; mouser# (none) -> 771-NTS0104GU12115
- IC306: Mfr. Texas Instruments -> (none); Mfr. No. DRV2603RUNT -> (none); Order Number 595-DRV2603RUNT -> (none); manf (none) -> Texas Instruments; manf# (none) -> DRV2603RUNT; mouser# (none) -> 595-DRV2603RUNT
- IC307: Mfr. Micro Crystal -> (none); Mfr. No. RV-8263-C8 32.768kHz-20PPM-TA-QA -> (none); Order Number 428-204291-MC01 -> (none); manf (none) -> Micro Crystal; manf# (none) -> RV-8263-C8 32.768kHz-20PPM-TA-QA; mouser# (none) -> 428-204291-MC01
- M301: Mfr. u-blox -> (none); Mfr. No. NORA-B106-00B -> (none); Order Number 377-NORA-B106-00B -> (none); manf (none) -> u-blox; manf# (none) -> NORA-B106-00B; mouser# (none) -> 377-NORA-B106-00B
- M302: Mfr. DFRobot -> (none); Mfr. No. FIT0774 -> (none); Order Number 426-FIT0774 -> (none); manf (none) -> DFRobot; manf# (none) -> FIT0774; mouser# (none) -> 426-FIT0774
- Q301: Mfr. Nexperia -> (none); Mfr. No. BC817W,115 -> (none); Order Number 771-BC817W115 -> (none); manf (none) -> Nexperia; manf# (none) -> BC817W,115; mouser# (none) -> 771-BC817W115
- Q302, Q303: Mfr. Nexperia -> (none); Mfr. No. PMZ550UNEYL -> (none); Order Number 771-PMZ550UNEYL -> (none); manf (none) -> Nexperia; manf# (none) -> PMZ550UNEYL; mouser# (none) -> 771-PMZ550UNEYL
- R301: Mfr. YAGEO -> (none); Mfr. No. RC0603FR-0712KL -> (none); Order Number 603-RC0603FR-0712KL -> (none); manf (none) -> YAGEO; manf# (none) -> RC0603FR-0712KL; mouser# (none) -> 603-RC0603FR-0712KL
- R302: Mfr. YAGEO -> (none); Mfr. No. RC0603FR-07100KL -> (none); Order Number 603-RC0603FR-07100KL -> (none); manf (none) -> YAGEO; manf# (none) -> RC0603FR-07100KL; mouser# (none) -> 603-RC0603FR-07100KL
- R303, R304: Mfr. YAGEO -> (none); Mfr. No. RC0603FR-074K7L -> (none); Order Number 603-RC0603FR-074K7L -> (none); manf (none) -> YAGEO; manf# (none) -> RC0603FR-074K7L; mouser# (none) -> 603-RC0603FR-074K7L
- R307: Mfr. YAGEO -> (none); Mfr. No. RC0603FR-07150KL -> (none); Order Number 603-RC0603FR-07150KL -> (none); manf (none) -> YAGEO; manf# (none) -> RC0603FR-07150KL; mouser# (none) -> 603-RC0603FR-07150KL
- R309, R313: Mfr. YAGEO -> (none); Mfr. No. RC0402FR-074K7L -> (none); Order Number 603-RC0402FR-074K7L -> (none); manf (none) -> YAGEO; manf# (none) -> RC0402FR-074K7L; mouser# (none) -> 603-RC0402FR-074K7L
- R311: Mfr. YAGEO -> (none); Mfr. No. RC0603FR-07180RL -> (none); Order Number 603-RC0603FR-07180RL -> (none); manf (none) -> YAGEO; manf# (none) -> RC0603FR-07180RL; mouser# (none) -> 603-RC0603FR-07180RL
- S301, S302, S303, S304: Mfr. E-Switch -> (none); Mfr. No. TL6340AF160Q -> (none); Order Number 612-TL6340AF160Q -> (none); manf (none) -> E-Switch; manf# (none) -> TL6340AF160Q; mouser# (none) -> 612-TL6340AF160Q
- X302: Mfr. EastRising -> (none); Mfr. No. OK-24F024-04 -> (none); manf (none) -> EastRising; manf# (none) -> OK-24F024-04
