File: hardware/ZSWatch.kicad_pcb (KiCad board)
At the start: 4 copper layers, 41 x 38 mm, 76 parts, among them IC101 nPM1300-QEXX, IC201 APDS-9306-065, IC202 BMI270, IC203 BMP581, IC204 LIS2MDLTR, IC302 FAN5622SX, IC303 MX25U51245GZ4I00, IC305 NTS0104GU12, IC306 DRV2603RUNT, IC307 RV-8263-C8, M301 NORA-B106, Q201 DMG1013UW-7, Q301 BC817W, Q302 PMZ550UNEYL, Q303 PMZ550UNEYL, X101 BATTERY, X302 GC9A01A_CST816S, X303 M+, X304 M-

Commit message: KiBot: Enhance KiBot configuration
- Implement #110
- Implement #109
- Add refresh for PCB specifications
- Add refresh for stackup

Signed-off-by: Daniel Kampert <danielkampert@kampis-elektroecke.de>
Other:
- board text added: "0,01 mm"
- board text added: "0,02"
- board text added: "0,035 mm"
- board text added: "0,1250 mm / 0,1250 mm"
- board text added: "0,196 mm"
- board text added: "0,2500 mm"
- board text added: "0,43 mm"
- board text added: "0,9820 mm"
- board text added: "3,3"
- board text added: "4,5"
- board text added: "40,9576 mm x 37,9989 mm"
- board text added: "Abmessungen der Platine:"
- board text added: "Castellated Pads:"
- board text added: "Dicke (mm)"
- board text added: "Dielektrikum"
- board text added: "Farbe"
- board text added: "Impedanzkontrolle:"
- board text added: "Kupferlagenanzahl:"
- board text added: "Kupferoberfläche:"
- board text added: "Lagenname"
- board text added: "Metallisierte Platinenkante:"
- board text added: "Min Leiterbahn/abstand:"
- board text added: "Min Lochdurchmesser:"
- board text added: "Nein"
- board text added: "PLATINEN-EIGENSCHAFTEN"
- board text added: "Platinen-Dicke:"
- board text added: "Randsteckverbinder:"
- board text added: "Tangens des Verlustwinkels"
- board text added: "Typ"
- board text removed: "0.01 mm"
- board text removed: "0.02"
- board text removed: "0.035 mm"
- board text removed: "0.1250 mm / 0.1250 mm"
- board text removed: "0.196 mm"
- board text removed: "0.2500 mm"
- board text removed: "0.43 mm"
- board text removed: "0.9820 mm"
- board text removed: "3.3"
- board text removed: "4.5"
- board text removed: "40.9576 mm x 37.9989 mm"
- board text removed: "BOARD CHARACTERISTICS"
- board text removed: "Board Thickness:"
- board text removed: "Board overall dimensions:"
- board text removed: "Castellated pads:"
- board text removed: "Color"
- board text removed: "Copper Finish:"
- board text removed: "Copper Layer Count:"
- board text removed: "Dielectric"
- board text removed: "Edge card connectors:"
- board text removed: "Impedance Control:"
- board text removed: "Layer Name"
- board text removed: "Loss Tangent"
- board text removed: "Min hole diameter:"
- board text removed: "Min track/spacing:"
- board text removed: "No"
- board text removed: "PCBWay 4-Layer Stack"
- board text removed: "Plated Board Edge:"
- board text removed: "Thickness (mm)"
- board text removed: "Type"
