File: dev-kit/Dev-Kit.kicad_sch (KiCad schematic)
At the start: 0 parts

Commit message: Cosmetic changes
Other:
- company: github.com/jakkra/ZSWatch-HW -> https://github.com/ZSWatch/Watch-HW
- title: https://github.com/ZSWatch/Watch-HW -> Watch-HW
