File: dev-kit/MCU.kicad_sch (KiCad schematic)
At the start: 34 parts, among them IC301 FAN5622SX, IC302 MX25U51245GZ4I00, IC303 USBLC6-2P6, IC304 NTS0104GU12, M301 NORA-B106, X301 Power, X302 Power, X303 Device, X304 UART, X305 IO Power, X306 Display, X307 Touch Power, X308 LED Power, X309 DEBUG, X310 GPIO

Commit message: Add impedance matching for USB, add jumper caps
Parts:
- added J301, J302, J303, J304: Jumper, symbol Misc:Jumper
- renumbered X310 to X304, X304 to X305, X305 to X306, X306 to X307, X307 to X308, X308 to X309, X309 to X310
Connections:
- net GND: now also R301.2; no longer R301.1
- net D+: now reaches IC303.1 (I/O1), X303.A6 (D+), X303.B6 (D+)
- net D-: now reaches IC303.3 (I/O2), X303.A7 (D-), X303.B7 (D-)
- net at IC301.3 (ISET): now also R301.1; no longer R301.2
Other:
- note added: "12k gives I_{LED} of <25 mA (max)"
- note removed: "NOTE: 12k gives I_{LED} of <25 mA (max)."
- title: ZSWatch v3 Dev-Kit -> https://github.com/ZSWatch/Watch-HW
- moved on the sheet: C301, IC301, R301, R303

Commit message: Cosmetic changes
Other:
- company: github.com/jakkra/ZSWatch-HW -> https://github.com/ZSWatch/Watch-HW
- title: https://github.com/ZSWatch/Watch-HW -> Watch-HW
Changed lines of the file:
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@@
 	(paper "A3")
 	(title_block
-		(title "https://github.com/ZSWatch/Watch-HW")
+		(title "Watch-HW")
 		(date "2025-05-09")
 		(rev "0")
-		(company "github.com/jakkra/ZSWatch-HW")
+		(company "https://github.com/ZSWatch/Watch-HW")
 	)
 	(text "From transmitter"

Commit message: Fix wrong part number
Parts:
- X303: manf# 12401610E4-2A -> 12401610E4#2A
Changed lines of the file:
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@@
 			)
 		)
-		(property "manf#" "12401610E4-2A"
+		(property "manf#" "12401610E4#2A"
 			(at 156.21 234.95 0)
 			(effects
