File: dev-kit/Peripherals.kicad_sch (KiCad schematic)
At the start: 49 parts, among them IC201 APDS-9306-065, IC202 RV-8263-C8, IC203 BMI270, IC204 LIS2MDLTR, IC205 BMP581, IC206 DRV2603RUNT, J201 Jumper, J202 Jumper, J203 Jumper, J204 Jumper, J205 Jumper, J206 Jumper, M201 Vibrator DC Motor, Q201 DMG1013UW-7, Q202 PMZ550UNEYL, Q203 PMZ550UNEYL, X201 Power, X202 I2S, X203 Power, X204 I2C, X205 Power, X206 Power, X207 Power, X208 Power, X209 Power, X210 Motor

Commit message: Fix wrong part numbers
Parts:
- R201: mouser# 603-RC0404FR-07150KL -> RC0402FR-07150KL
- R202, R203: manf# RC0402FR-074K7L -> RC0402FR-071K8L; mouser# 603-RC0402FR-074K7L -> 603-RC0402FR-071K8L
Changed lines of the file:
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@@
 			)
 		)
-		(property "mouser#" "603-RC0404FR-07150KL"
+		(property "mouser#" "RC0402FR-07150KL"
 			(at 76.2 233.68 0)
 			(effects
@@
 			)
 		)
-		(property "manf#" "RC0402FR-074K7L"
+		(property "manf#" "RC0402FR-071K8L"
 			(at 142.24 261.62 0)
 			(effects
@@
 			)
 		)
-		(property "mouser#" "603-RC0402FR-074K7L"
+		(property "mouser#" "603-RC0402FR-071K8L"
 			(at 142.24 261.62 0)
 			(effects
@@
 			)
 		)
-		(property "manf#" "RC0402FR-074K7L"
+		(property "manf#" "RC0402FR-071K8L"
 			(at 142.24 236.22 0)
 			(effects
@@
 			)
 		)
-		(property "mouser#" "603-RC0402FR-074K7L"
+		(property "mouser#" "603-RC0402FR-071K8L"
 			(at 142.24 236.22 0)
 			(effects
