File: dev-kit/Power.kicad_sch (KiCad schematic)
At the start: 26 parts, among them IC101 nPM1300-QEXX, X101 Battery, X102 Battery, X103 Power

Commit message: Fix wrong part numbers
Parts:
- C103: manf# 04026D105MAT4A -> 0402ZD225MAT2A; mouser# 581-04026D105MAT4A -> 581-0402ZD225MAT2A
- R102: mouser# 603-RC0402FR-07150KL -> RC0402FR-07150KL
Changed lines of the file:
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@@
 			)
 		)
-		(property "mouser#" "603-RC0402FR-07150KL"
+		(property "mouser#" "RC0402FR-07150KL"
 			(at 82.55 134.62 0)
 			(effects
@@
 			)
 		)
-		(property "manf#" "04026D105MAT4A"
+		(property "manf#" "0402ZD225MAT2A"
 			(at 140.97 44.45 0)
 			(effects
@@
 			)
 		)
-		(property "mouser#" "581-04026D105MAT4A"
+		(property "mouser#" "581-0402ZD225MAT2A"
 			(at 140.97 44.45 0)
 			(effects
